File: ATtiny-313.sch (EAGLE design)
At the start: 13 parts

Commit message: use SMD to tighten up design
Parts:
- removed LED1: (no value), SparkFun-LED:LED5MM
- removed R1: 68, resistor:R-US_0207/10
- added LED2: (no value), led:LEDSMT1206
- added R2: 680, resistor:R-US_R3216
Connections:
- net N$2: now also LED2.A; no longer LED1.A
- net N$24: now also LED2.C, R2.2; no longer LED1.C, R1.2
- net N$3: now also R2.1; no longer R1.1
Changed lines of the file:
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@@
 <part name="JP3" library="pinhead" deviceset="PINHD-1X10" device=""/>
 <part name="JP6" library="pinhead" deviceset="PINHD-1X3" device=""/>
-<part name="LED1" library="SparkFun-LED" deviceset="LED" device="5MM"/>
-<part name="R1" library="resistor" deviceset="R-US_" device="0207/10" value="68"/>
 <part name="ISP" library="pinhead" deviceset="PINHD-2X3" device=""/>
 <part name="S1" library="switch-omron" deviceset="10-XX" device=""/>
 <part name="JP4" library="pinhead" deviceset="PINHD-1X1" device=""/>
+<part name="LED2" library="led" deviceset="LED" device="SMT1206"/>
+<part name="R2" library="resistor" deviceset="R-US_" device="R3216" value="680"/>
 </parts>
 <sheets>
@@
 <instance part="JP3" gate="A" x="127" y="7.62"/>
 <instance part="JP6" gate="A" x="99.06" y="53.34"/>
-<instance part="LED1" gate="G$1" x="78.74" y="35.56" rot="R270"/>
-<instance part="R1" gate="G$1" x="63.5" y="35.56"/>
 <instance part="ISP" gate="A" x="111.76" y="76.2"/>
 <instance part="S1" gate="1" x="35.56" y="30.48"/>
 <instance part="JP4" gate="G$1" x="17.78" y="71.12"/>
+<instance part="LED2" gate="G$1" x="78.74" y="35.56" rot="R270"/>
+<instance part="R2" gate="G$1" x="63.5" y="35.56"/>
 </instances>
 <busses>
@@
 <wire x1="86.36" y1="53.34" x2="96.52" y2="53.34" width="0.1524" layer="91"/>
 <junction x="96.52" y="53.34"/>
-<pinref part="LED1" gate="G$1" pin="A"/>
 <wire x1="86.36" y1="35.56" x2="81.28" y2="35.56" width="0.1524" layer="91"/>
+<junction x="86.36" y="35.56"/>
+<pinref part="LED2" gate="G$1" pin="A"/>
 <junction x="81.28" y="35.56"/>
-<junction x="86.36" y="35.56"/>
 </segment>
 </net>
@@
 <junction x="43.18" y="-5.08"/>
 <junction x="5.08" y="-5.08"/>
-<pinref part="R1" gate="G$1" pin="1"/>
 <wire x1="58.42" y1="35.56" x2="55.88" y2="35.56" width="0.1524" layer="91"/>
 <wire x1="55.88" y1="35.56" x2="55.88" y2="40.64" width="0.1524" layer="91"/>
 <junction x="55.88" y="40.64"/>
-<junction x="58.42" y="35.56"/>
 <wire x1="68.58" y1="40.64" x2="129.54" y2="40.64" width="0.1524" layer="91"/>
 <wire x1="129.54" y1="40.64" x2="129.54" y2="73.66" width="0.1524" layer="91"/>
@@
 <junction x="35.56" y="35.56"/>
 <junction x="35.56" y="40.64"/>
+<pinref part="R2" gate="G$1" pin="1"/>
+<junction x="58.42" y="35.56"/>
 </segment>
 </net>
@@
 <net name="N$24" class="0">
 <segment>
-<pinref part="LED1" gate="G$1" pin="C"/>
-<pinref part="R1" gate="G$1" pin="2"/>
 <wire x1="68.58" y1="35.56" x2="73.66" y2="35.56" width="0.1524" layer="91"/>
+<pinref part="R2" gate="G$1" pin="2"/>
+<pinref part="LED2" gate="G$1" pin="C"/>
 <junction x="68.58" y="35.56"/>
 <junction x="73.66" y="35.56"/>

Commit message: more SMD goodness
Parts:
- removed U$1: V_REG_LD1117VXX, SparkFun-PowerIC:V_REG_LD1117VXX
- added IC1: REG1117, burr-brown:REG1117
Connections:
- net N$1: now also IC1.VIN; no longer U$1.IN
- net N$3: now also IC1.GND; no longer U$1.GND
- net N$4: now also IC1.VOUT; no longer U$1.OUT
Changed lines of the file:
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@@
 <part name="ATTINY2313" library="ic-package" deviceset="DIL20" device="S"/>
 <part name="JP1" library="SparkFun-Connectors" deviceset="USB" device="PTH" value="USB-B"/>
-<part name="U$1" library="SparkFun-PowerIC" deviceset="V_REG_LD1117VXX" device=""/>
 <part name="C1" library="rcl" deviceset="CPOL-US" device="E1.8-4" value="10 uF"/>
 <part name="C2" library="rcl" deviceset="CPOL-US" device="E1.8-4" value="10 uF"/>
@@
 <part name="LED2" library="led" deviceset="LED" device="SMT1206"/>
 <part name="R2" library="resistor" deviceset="R-US_" device="R3216" value="680"/>
+<part name="IC1" library="burr-brown" deviceset="REG1117" device=""/>
 </parts>
 <sheets>
@@
 <instance part="ATTINY2313" gate="G$1" x="60.96" y="7.62"/>
 <instance part="JP1" gate="G$1" x="25.4" y="83.82" rot="R90"/>
-<instance part="U$1" gate="G$1" x="48.26" y="68.58"/>
 <instance part="C1" gate="G$1" x="68.58" y="48.26" rot="R180"/>
 <instance part="C2" gate="G$1" x="33.02" y="58.42" rot="R180"/>
@@
 <instance part="LED2" gate="G$1" x="78.74" y="35.56" rot="R270"/>
 <instance part="R2" gate="G$1" x="63.5" y="35.56"/>
+<instance part="IC1" gate="G$1" x="53.34" y="68.58"/>
 </instances>
 <busses>
@@
 <wire x1="22.86" y1="68.58" x2="30.48" y2="68.58" width="0.1524" layer="91"/>
 <wire x1="30.48" y1="68.58" x2="33.02" y2="68.58" width="0.1524" layer="91"/>
-<pinref part="U$1" gate="G$1" pin="IN"/>
-<wire x1="33.02" y1="68.58" x2="35.56" y2="68.58" width="0.1524" layer="91"/>
-<wire x1="35.56" y1="68.58" x2="40.64" y2="68.58" width="0.1524" layer="91"/>
+<wire x1="33.02" y1="68.58" x2="38.1" y2="68.58" width="0.1524" layer="91"/>
 <junction x="22.86" y="81.28"/>
-<junction x="40.64" y="68.58"/>
 <pinref part="C2" gate="G$1" pin="-"/>
 <wire x1="33.02" y1="63.5" x2="33.02" y2="68.58" width="0.1524" layer="91"/>
@@
 <junction x="22.86" y="71.12"/>
 <junction x="15.24" y="71.12"/>
+<pinref part="IC1" gate="G$1" pin="VIN"/>
+<wire x1="38.1" y1="68.58" x2="40.64" y2="68.58" width="0.1524" layer="91"/>
+<junction x="40.64" y="68.58"/>
 </segment>
 </net>
@@
 <wire x1="35.56" y1="40.64" x2="43.18" y2="40.64" width="0.1524" layer="91"/>
 <wire x1="43.18" y1="40.64" x2="48.26" y2="40.64" width="0.1524" layer="91"/>
-<wire x1="48.26" y1="40.64" x2="55.88" y2="40.64" width="0.1524" layer="91"/>
+<wire x1="48.26" y1="40.64" x2="53.34" y2="40.64" width="0.1524" layer="91"/>
+<wire x1="53.34" y1="40.64" x2="55.88" y2="40.64" width="0.1524" layer="91"/>
 <wire x1="55.88" y1="40.64" x2="68.58" y2="40.64" width="0.1524" layer="91"/>
 <wire x1="68.58" y1="40.64" x2="68.58" y2="45.72" width="0.1524" layer="91"/>
-<pinref part="U$1" gate="G$1" pin="GND"/>
-<wire x1="48.26" y1="60.96" x2="48.26" y2="40.64" width="0.1524" layer="91"/>
-<junction x="48.26" y="60.96"/>
-<junction x="48.26" y="40.64"/>
 <junction x="68.58" y="45.72"/>
 <junction x="33.02" y="55.88"/>
@@
 <pinref part="R2" gate="G$1" pin="1"/>
 <junction x="58.42" y="35.56"/>
+<pinref part="IC1" gate="G$1" pin="GND"/>
+<wire x1="53.34" y1="55.88" x2="53.34" y2="40.64" width="0.1524" layer="91"/>
+<junction x="53.34" y="40.64"/>
+<junction x="53.34" y="55.88"/>
 </segment>
 </net>
@@
 <segment>
 <pinref part="C1" gate="G$1" pin="-"/>
-<pinref part="U$1" gate="G$1" pin="OUT"/>
-<junction x="55.88" y="68.58"/>
-<wire x1="55.88" y1="68.58" x2="68.58" y2="68.58" width="0.1524" layer="91"/>
 <wire x1="68.58" y1="68.58" x2="91.44" y2="68.58" width="0.1524" layer="91"/>
-<junction x="68.58" y="68.58"/>
 <wire x1="68.58" y1="68.58" x2="68.58" y2="53.34" width="0.1524" layer="91"/>
 <junction x="68.58" y="53.34"/>
@@
 <junction x="96.52" y="55.88"/>
 <junction x="91.44" y="68.58"/>
-</segment>
-</net>
+<pinref part="IC1" gate="G$1" pin="VOUT"/>
+<wire x1="68.58" y1="68.58" x2="66.04" y2="68.58" width="0.1524" layer="91"/>
+<junction x="68.58" y="68.58"/>
+<junction x="66.04" y="68.58"/>
+</segment>
+</net>

Commit message: tightened up the design
Parts:
- removed JP6: (no value), pinhead:PINHD-1X3
Connections:
- net ISP renamed MISO'
- net N$1 renamed 5V
- net N$14 renamed SCLK'
- net N$16 renamed MOSI'
- net N$3 renamed GND
- net N$5 renamed REST'
- removed net N$2: ATTINY2313.20, JP3.1, JP6.2, LED2.A
- removed net N$23: ISP.2, JP6.3
- removed net N$4: C1.-, IC1.VOUT, JP6.1
- new net 3.3V: ATTINY2313.20, C1.-, IC1.VOUT, JP3.1, LED2.A
Other:
- note added: "MISO'"
- note added: "MOSI'"
- note added: "REST'"
- note added: "SCLK'"
- moved on the sheet: C1, JP4, LED2, R2, S1

Commit message: added built in ISP
Parts:
- removed ISP: (no value), pinhead:PINHD-2X3
- added D3, D4: 3.6V, .5W, diode:ZENER-DIODEDO35Z10
- added IC2: ATtiny85, ic-package:DIL8
- added R1, R3: 68, resistor:R-US_R3216
- added R4: 1.5K, resistor:R-US_R3216
Connections:
- new net D+': D4.C, JP1.D+, R1.2
- new net D-': D3.C, JP1.D-, R3.2, R4.1
- new net N$1: IC2.2, R1.1
- new net N$2: IC2.3, R3.1
- net 5V: now also IC2.8, R4.2
- net GND: now also D3.A, D4.A, IC2.4; no longer ISP.6
- net MISO': now also IC2.6; no longer ISP.1
- net MOSI': now also IC2.5; no longer ISP.4
- net REST': now also IC2.1; no longer ISP.5
- net SCLK': now also IC2.7; no longer ISP.3
Other:
- note added: "D+'"
- note added: "D-'"
Changed lines of the file:
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@@
 <part name="JP2" library="pinhead" deviceset="PINHD-1X10" device=""/>
 <part name="JP3" library="pinhead" deviceset="PINHD-1X10" device=""/>
-<part name="ISP" library="pinhead" deviceset="PINHD-2X3" device=""/>
 <part name="S1" library="switch-omron" deviceset="10-XX" device=""/>
 <part name="JP4" library="pinhead" deviceset="PINHD-1X1" device=""/>
@@
 <part name="SUPPLY6" library="SparkFun-Aesthetics" deviceset="5V" device=""/>
 <part name="SUPPLY7" library="SparkFun-Aesthetics" deviceset="5V" device=""/>
+<part name="IC2" library="ic-package" deviceset="DIL8" device="" value="ATtiny85"/>
+<part name="R1" library="resistor" deviceset="R-US_" device="R3216" value="68"/>
+<part name="R3" library="resistor" deviceset="R-US_" device="R3216" value="68"/>
+<part name="R4" library="resistor" deviceset="R-US_" device="R3216" value="1.5K"/>
+<part name="SUPPLY8" library="SparkFun-Aesthetics" deviceset="5V" device=""/>
+<part name="GND10" library="SparkFun-Aesthetics" deviceset="GND" device=""/>
+<part name="SUPPLY9" library="SparkFun-Aesthetics" deviceset="5V" device=""/>
+<part name="GND11" library="SparkFun-Aesthetics" deviceset="GND" device=""/>
+<part name="D3" library="diode" deviceset="ZENER-DIODE" device="DO35Z10" value="3.6V, .5W"/>
+<part name="D4" library="diode" deviceset="ZENER-DIODE" device="DO35Z10" value="3.6V, .5W"/>
 </parts>
 <sheets>
@@
 <plain>
 <text x="48.26" y="22.86" size="1.778" layer="95" rot="R90">REST'</text>
-<text x="99.06" y="76.2" size="1.778" layer="95" rot="R180">REST'</text>
-<text x="99.06" y="76.2" size="1.778" layer="95" rot="R180">REST'</text>
+<text x="106.68" y="68.58" size="1.778" layer="95" rot="R270">REST'</text>
 <text x="-17.78" y="38.1" size="1.778" layer="95" rot="R90">REST'</text>
 <text x="10.16" y="17.78" size="1.778" layer="95">REST'</text>
-<text x="83.82" y="76.2" size="1.778" layer="95">SCLK'</text>
+<text x="124.46" y="55.88" size="1.778" layer="95">SCLK'</text>
 <text x="73.66" y="15.24" size="1.778" layer="95">SCLK'</text>
 <text x="111.76" y="15.24" size="1.778" layer="95">SCLK'</text>
-<text x="99.06" y="78.74" size="1.778" layer="95">MISO'</text>
+<text x="124.46" y="53.34" size="1.778" layer="95">MISO'</text>
 <text x="73.66" y="12.7" size="1.778" layer="95">MISO'</text>
 <text x="111.76" y="12.7" size="1.778" layer="95">MISO'</text>
-<text x="124.46" y="76.2" size="1.778" layer="95">MOSI'</text>
+<text x="124.46" y="50.8" size="1.778" layer="95">MOSI'</text>
 <text x="73.66" y="10.16" size="1.778" layer="95">MOSI'</text>
 <text x="111.76" y="10.16" size="1.778" layer="95">MOSI'</text>
+<text x="78.74" y="53.34" size="1.778" layer="95">D-'</text>
+<text x="101.6" y="71.12" size="1.778" layer="95" rot="R90">D+'</text>
 </plain>
 <instances>
@@
 <instance part="JP2" gate="A" x="7.62" y="7.62"/>
 <instance part="JP3" gate="A" x="127" y="7.62"/>
-<instance part="ISP" gate="A" x="111.76" y="76.2"/>
 <instance part="S1" gate="1" x="-20.32" y="50.8"/>
 <instance part="JP4" gate="G$1" x="5.08" y="66.04" rot="R90"/>
@@
 <instance part="GND4" gate="1" x="53.34" y="50.8"/>
 <instance part="GND5" gate="1" x="68.58" y="50.8"/>
-<instance part="GND6" gate="1" x="129.54" y="68.58"/>
+<instance part="GND6" gate="1" x="104.14" y="45.72"/>
 <instance part="GND7" gate="1" x="48.26" y="-5.08" rot="R270"/>
 <instance part="GND8" gate="1" x="12.7" y="-5.08" rot="R90"/>
@@
 <instance part="SUPPLY6" gate="G$1" x="5.08" y="68.58"/>
 <instance part="SUPPLY7" gate="G$1" x="30.48" y="68.58" rot="R90"/>
+<instance part="IC2" gate="G$1" x="114.3" y="55.88"/>
+<instance part="R1" gate="G$1" x="101.6" y="60.96" rot="R90"/>
+<instance part="R3" gate="G$1" x="91.44" y="53.34" rot="R180"/>
+<instance part="R4" gate="G$1" x="86.36" y="63.5" rot="R90"/>
+<instance part="SUPPLY8" gate="G$1" x="124.46" y="60.96"/>
+<instance part="GND10" gate="1" x="86.36" y="38.1"/>
+<instance part="SUPPLY9" gate="G$1" x="86.36" y="71.12"/>
+<instance part="GND11" gate="1" x="93.98" y="71.12" rot="R180"/>
+<instance part="D3" gate="G$1" x="86.36" y="45.72" rot="R90"/>
+<instance part="D4" gate="G$1" x="96.52" y="66.04"/>
 </instances>
 <busses>
@@
 <net name="MOSI'" class="0">
 <segment>
-<pinref part="ISP" gate="A" pin="4"/>
-<wire x1="116.84" y1="76.2" x2="129.54" y2="76.2" width="0.1524" layer="91"/>
-<junction x="116.84" y="76.2"/>
+<wire x1="121.92" y1="50.8" x2="127" y2="50.8" width="0.1524" layer="91"/>
+<pinref part="IC2" gate="G$1" pin="5"/>
+<junction x="121.92" y="50.8"/>
 </segment>
 <segment>
@@
 </segment>
 <segment>
-<wire x1="129.54" y1="71.12" x2="129.54" y2="73.66" width="0.1524" layer="91"/>
-<pinref part="ISP" gate="A" pin="6"/>
-<wire x1="129.54" y1="73.66" x2="116.84" y2="73.66" width="0.1524" layer="91"/>
-<junction x="116.84" y="73.66"/>
+<wire x1="104.14" y1="48.26" x2="104.14" y2="50.8" width="0.1524" layer="91"/>
+<wire x1="104.14" y1="50.8" x2="106.68" y2="50.8" width="0.1524" layer="91"/>
 <pinref part="GND6" gate="1" pin="GND"/>
+<pinref part="IC2" gate="G$1" pin="4"/>
+<junction x="106.68" y="50.8"/>
+</segment>
+<segment>
+<pinref part="GND10" gate="1" pin="GND"/>
+<wire x1="86.36" y1="40.64" x2="86.36" y2="43.18" width="0.1524" layer="91"/>
+<junction x="86.36" y="40.64"/>
+<pinref part="D3" gate="G$1" pin="A"/>
+<junction x="86.36" y="43.18"/>
+</segment>
+<segment>
+<pinref part="GND11" gate="1" pin="GND"/>
+<wire x1="93.98" y1="68.58" x2="93.98" y2="66.04" width="0.1524" layer="91"/>
+<junction x="93.98" y="68.58"/>
+<pinref part="D4" gate="G$1" pin="A"/>
+<junction x="93.98" y="66.04"/>
 </segment>
 </net>
@@
 <wire x1="22.86" y1="78.74" x2="22.86" y2="81.28" width="0.1524" layer="91"/>
 </segment>
+<segment>
+<pinref part="IC2" gate="G$1" pin="8"/>
+<wire x1="121.92" y1="58.42" x2="124.46" y2="58.42" width="0.1524" layer="91"/>
+<pinref part="SUPPLY8" gate="G$1" pin="5V"/>
+<wire x1="124.46" y1="58.42" x2="124.46" y2="60.96" width="0.1524" layer="91"/>
+<junction x="121.92" y="58.42"/>
+<junction x="124.46" y="60.96"/>
+</segment>
+<segment>
+<pinref part="SUPPLY9" gate="G$1" pin="5V"/>
+<pinref part="R4" gate="G$1" pin="2"/>
+<wire x1="86.36" y1="71.12" x2="86.36" y2="68.58" width="0.1524" layer="91"/>
+<junction x="86.36" y="71.12"/>
+<junction x="86.36" y="68.58"/>
+</segment>
 </net>
 <net name="REST'" class="0">
 <segment>
-<pinref part="ISP" gate="A" pin="5"/>
-<junction x="109.22" y="73.66"/>
-<wire x1="91.44" y1="73.66" x2="109.22" y2="73.66" width="0.1524" layer="91"/>
+<wire x1="106.68" y1="66.04" x2="106.68" y2="58.42" width="0.1524" layer="91"/>
+<pinref part="IC2" gate="G$1" pin="1"/>
+<junction x="106.68" y="58.42"/>
 </segment>
 <segment>
@@
 <net name="SCLK'" class="0">
 <segment>
-<pinref part="ISP" gate="A" pin="3"/>
-<junction x="109.22" y="76.2"/>
-<wire x1="101.6" y1="76.2" x2="109.22" y2="76.2" width="0.1524" layer="91"/>
-<wire x1="101.6" y1="76.2" x2="83.82" y2="76.2" width="0.1524" layer="91"/>
+<wire x1="127" y1="55.88" x2="121.92" y2="55.88" width="0.1524" layer="91"/>
+<pinref part="IC2" gate="G$1" pin="7"/>
+<junction x="121.92" y="55.88"/>
 </segment>
 <segment>
@@
 <net name="MISO'" class="0">
 <segment>
-<pinref part="ISP" gate="A" pin="1"/>
-<junction x="109.22" y="78.74"/>
-<wire x1="99.06" y1="78.74" x2="109.22" y2="78.74" width="0.1524" layer="91"/>
+<wire x1="127" y1="53.34" x2="121.92" y2="53.34" width="0.1524" layer="91"/>
+<pinref part="IC2" gate="G$1" pin="6"/>
+<junction x="121.92" y="53.34"/>
 </segment>
 <segment>
@@
 </segment>
 </net>
+<net name="N$2" class="0">
+<segment>
+<pinref part="IC2" gate="G$1" pin="3"/>
+<pinref part="R3" gate="G$1" pin="1"/>
+<wire x1="106.68" y1="53.34" x2="96.52" y2="53.34" width="0.1524" layer="91"/>
+<junction x="96.52" y="53.34"/>
+<junction x="106.68" y="53.34"/>
+</segment>
+</net>
+<net name="D-'" class="0">
+<segment>
+<pinref part="JP1" gate="G$1" pin="D-"/>
+<wire x1="20.32" y1="81.28" x2="20.32" y2="76.2" width="0.1524" layer="91"/>
+</segment>
+<segment>
+<pinref part="R3" gate="G$1" pin="2"/>
+<wire x1="86.36" y1="48.26" x2="86.36" y2="53.34" width="0.1524" layer="91"/>
+<junction x="86.36" y="53.34"/>
+<wire x1="86.36" y1="53.34" x2="78.74" y2="53.34" width="0.1524" layer="91"/>
+<pinref part="R4" gate="G$1" pin="1"/>
+<wire x1="86.36" y1="53.34" x2="86.36" y2="58.42" width="0.1524" layer="91"/>
+<junction x="86.36" y="58.42"/>
+<pinref part="D3" gate="G$1" pin="C"/>
+<junction x="86.36" y="48.26"/>
+</segment>
+</net>
+<net name="D+'" class="0">
+<segment>
+<pinref part="JP1" gate="G$1" pin="D+"/>
+<wire x1="17.78" y1="81.28" x2="17.78" y2="76.2" width="0.1524" layer="91"/>
+</segment>
+<segment>
+<pinref part="R1" gate="G$1" pin="2"/>
+<wire x1="99.06" y1="66.04" x2="101.6" y2="66.04" width="0.1524" layer="91"/>
+<junction x="101.6" y="66.04"/>
+<wire x1="101.6" y1="66.04" x2="101.6" y2="73.66" width="0.1524" layer="91"/>
+<pinref part="D4" gate="G$1" pin="C"/>
+<junction x="99.06" y="66.04"/>
+</segment>
+</net>
+<net name="N$1" class="0">
+<segment>
+<pinref part="IC2" gate="G$1" pin="2"/>
+<pinref part="R1" gate="G$1" pin="1"/>
+<wire x1="106.68" y1="55.88" x2="101.6" y2="55.88" width="0.1524" layer="91"/>
+<junction x="106.68" y="55.88"/>
+<junction x="101.6" y="55.88"/>
+</segment>
+</net>
